Commit message: Gazebo launch script added...debugging gazebo_control

File: description/cy-borg.urdf.xacro (robot description, xacro)
@@ -3,3 +3,4 @@
     <!-- Chassis-->
     <xacro:include filename="cy-borg_core.xacro" />
+    <xacro:include filename="gazebo_control.xacro" />
 </robot>

File: description/cy-borg_core.xacro (robot description, xacro)
@@ -16,4 +16,5 @@
     <!--BASE LINK-->
     <link name="base_link">
+    <origin xyz="0 0 0.5" />
     </link>
     <!--CHASSIS LINK-->

Commit message: pre install folder cleaning

File: description/cy-borg.urdf.xacro (robot description, xacro)
@@ -3,4 +3,5 @@
     <!-- Chassis-->
     <xacro:include filename="cy-borg_core.xacro" />
-    <xacro:include filename="gazebo_control.xacro" />
+    <!--<xacro:include filename="gazebo_control.xacro" />-->
+    <xacro:include filename="ros2_control.xacro" />
 </robot>

File: description/cy-borg_core.xacro (robot description, xacro)
@@ -16,5 +16,5 @@
     <!--BASE LINK-->
     <link name="base_link">
-    <origin xyz="0 0 0.5" />
+        <origin xyz="0 0 0.5" />
     </link>
     <!--CHASSIS LINK-->
